File: PCB/mcus.kicad_sch (KiCad schematic)
At the start: 62 parts, among them SW1 SW_Push, SW2 SW_Push, U1 APS6404L-SQN-SN, U21 W25Q128JVS, U24 RP2350A, U25 W25Q128JVS, U27 RP2350A, Y4 ABM8-272-T3, Y5 ABM8-272-T3

Commit message: Fix MPN number, adjust footprint, production files
Parts:
- SW1, SW2: MPN (none) -> TS-1088-AR02016
Changed lines of the file:
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@@
 			)
 		)
+		(property "MPN" "TS-1088-AR02016"
+			(at 146.05 60.96 0)
+			(hide yes)
+			(show_name no)
+			(do_not_autoplace no)
+			(effects
+				(font
+					(size 1.27 1.27)
+				)
+			)
+		)
 		(pin "2"
 		)
@@
 			(at 146.05 85.09 0)
 			(hide yes)
+			(show_name no)
+			(do_not_autoplace no)
+			(effects
+				(font
+					(size 1.27 1.27)
+				)
+			)
+		)
+		(property "MPN" "TS-1088-AR02016"
+			(at 146.05 85.09 0)
+			(hide yes)
